File: tpa3116_amplifier_board.kicad_pcb (KiCad board)
At the start: 2 copper layers, 60.3 x 50.8 mm, 41 parts, among them IC1 TPA3116D2QDADRQ1, J1 power_supply, J2 Conn_01x04, J3 power_supply, J4 output_right

Commit message: мелкие правки
Routing:
- net VCC: track 71.2 -> 71.4 mm, vias 19 -> 18
- net GND: vias 93 -> 94
Changed lines of the file:
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@@
     (property "ki_keywords" "cap capacitor")
     (attr smd)
-    (fp_text reference "C3" (at -2.54 0 90) (layer "F.SilkS")
+    (fp_text reference "C3" (at 2.8575 0 90) (layer "F.SilkS")
         (effects (font (size 1 1) (thickness 0.15)))
     )
@@
     (height -13.335)
     (gr_text "60,3250 mm" (at 131.1275 80.13) (layer "Dwgs.User")
+      (effects (font (size 1 1) (thickness 0.15)))
+    )
+    (format (prefix "") (suffix "") (units 3) (units_format 1) (precision 4))
+    (style (thickness 0.1) (arrow_length 1.27) (text_position_mode 0) (extension_height 0.58642) (extension_offset 0.5) keep_text_aligned)
+  )
+  (dimension (type aligned) (layer "Dwgs.User")
+    (pts (xy 124.46 100) (xy 124.46 140))
+    (height 40.005)
+    (gr_text "40,0000 mm" (at 83.305 120 90) (layer "Dwgs.User")
       (effects (font (size 1 1) (thickness 0.15)))
     )
@@
   (via (at 123.19 114.935) (size 0.8) (drill 0.4) (layers "F.Cu" "B.Cu") (free) (net 5))
   (via (at 152.4 102.87) (size 0.8) (drill 0.4) (layers "F.Cu" "B.Cu") (free) (net 5))
-  (via (at 111.252 125.476) (size 0.8) (drill 0.4) (layers "F.Cu" "B.Cu") (free) (net 5))
+  (via (at 111.76 123.825) (size 0.8) (drill 0.4) (layers "F.Cu" "B.Cu") (free) (net 5))
   (via (at 121.263 113.665) (size 0.8) (drill 0.4) (layers "F.Cu" "B.Cu") (free) (net 5))
   (via (at 137.03 121.92) (size 0.8) (drill 0.4) (layers "F.Cu" "B.Cu") (free) (net 5))
@@
   (via (at 121.263 130.175) (size 0.8) (drill 0.4) (layers "F.Cu" "B.Cu") (free) (net 5))
   (via (at 124.46 123.825) (size 0.8) (drill 0.4) (layers "F.Cu" "B.Cu") (free) (net 5))
-  (via (at 108.204 116.84) (size 0.8) (drill 0.4) (layers "F.Cu" "B.Cu") (free) (net 5))
+  (via (at 109.22 116.84) (size 0.8) (drill 0.4) (layers "F.Cu" "B.Cu") (free) (net 5))
   (via (at 124.46 116.205) (size 0.8) (drill 0.4) (layers "F.Cu" "B.Cu") (free) (net 5))
+  (via (at 106.68 123.825) (size 0.8) (drill 0.4) (layers "F.Cu" "B.Cu") (free) (net 5))
   (via (at 128.27 142.875) (size 0.8) (drill 0.4) (layers "F.Cu" "B.Cu") (free) (net 5))
   (via (at 133.35 142.875) (size 0.8) (drill 0.4) (layers "F.Cu" "B.Cu") (free) (net 5))
@@
   (via (at 124.46 125.095) (size 0.8) (drill 0.4) (layers "F.Cu" "B.Cu") (free) (net 5))
   (via (at 142.24 107.95) (size 0.8) (drill 0.4) (layers "F.Cu" "B.Cu") (free) (net 5))
-  (via (at 111.252 127.508) (size 0.8) (drill 0.4) (layers "F.Cu" "B.Cu") (free) (net 5))
+  (via (at 111.76 127.635) (size 0.8) (drill 0.4) (layers "F.Cu" "B.Cu") (free) (net 5))
   (via (at 128.27 107.315) (size 0.8) (drill 0.4) (layers "F.Cu" "B.Cu") (free) (net 5))
   (via (at 124.46 117.475) (size 0.8) (drill 0.4) (layers "F.Cu" "B.Cu") (free) (net 5))
@@
   (via (at 122.533 111.125) (size 0.8) (drill 0.4) (layers "F.Cu" "B.Cu") (free) (net 5))
   (via (at 121.263 128.905) (size 0.8) (drill 0.4) (layers "F.Cu" "B.Cu") (free) (net 5))
-  (via (at 106.045 118.745) (size 0.8) (drill 0.4) (layers "F.Cu" "B.Cu") (free) (net 5))
+  (via (at 106.68 119.38) (size 0.8) (drill 0.4) (layers "F.Cu" "B.Cu") (free) (net 5))
   (via (at 142.24 132.08) (size 0.8) (drill 0.4) (layers "F.Cu" "B.Cu") (free) (net 5))
   (via (at 147.32 134.62) (size 0.8) (drill 0.4) (layers "F.Cu" "B.Cu") (free) (net 5))
@@
   (via (at 113.03 97.155) (size 0.8) (drill 0.4) (layers "F.Cu" "B.Cu") (free) (net 5))
   (via (at 124.46 122.555) (size 0.8) (drill 0.4) (layers "F.Cu" "B.Cu") (free) (net 5))
-  (via (at 106.045 116.84) (size 0.8) (drill 0.4) (layers "F.Cu" "B.Cu") (free) (net 5))
   (via (at 125.73 123.825) (size 0.8) (drill 0.4) (layers "F.Cu" "B.Cu") (free) (net 5))
   (via (at 149.86 139.7) (size 0.8) (drill 0.4) (layers "F.Cu" "B.Cu") (free) (net 5))
-  (via (at 107.188 127.508) (size 0.8) (drill 0.4) (layers "F.Cu" "B.Cu") (free) (net 5))
+  (via (at 106.68 127.635) (size 0.8) (drill 0.4) (layers "F.Cu" "B.Cu") (free) (net 5))
   (via (at 118.11 142.875) (size 0.8) (drill 0.4) (layers "F.Cu" "B.Cu") (free) (net 5))
   (via (at 144.78 107.95) (size 0.8) (drill 0.4) (layers "F.Cu" "B.Cu") (free) (net 5))
   (via (at 124.46 114.935) (size 0.8) (drill 0.4) (layers "F.Cu" "B.Cu") (free) (net 5))
-  (via (at 109.22 127.508) (size 0.8) (drill 0.4) (layers "F.Cu" "B.Cu") (free) (net 5))
+  (via (at 109.22 127.635) (size 0.8) (drill 0.4) (layers "F.Cu" "B.Cu") (free) (net 5))
   (via (at 123.19 116.205) (size 0.8) (drill 0.4) (layers "F.Cu" "B.Cu") (free) (net 5))
+  (via (at 153.035 95.885) (size 0.8) (drill 0.4) (layers "F.Cu" "B.Cu") (free) (net 5))
   (via (at 123.19 125.095) (size 0.8) (drill 0.4) (layers "F.Cu" "B.Cu") (free) (net 5))
   (via (at 122.533 126.365) (size 0.8) (drill 0.4) (layers "F.Cu" "B.Cu") (free) (net 5))
   (via (at 144.78 105.41) (size 0.8) (drill 0.4) (layers "F.Cu" "B.Cu") (free) (net 5))
-  (via (at 109.22 125.476) (size 0.8) (drill 0.4) (layers "F.Cu" "B.Cu") (free) (net 5))
+  (via (at 109.22 123.825) (size 0.8) (drill 0.4) (layers "F.Cu" "B.Cu") (free) (net 5))
   (via (at 122.533 127.635) (size 0.8) (drill 0.4) (layers "F.Cu" "B.Cu") (free) (net 5))
   (via (at 121.263 109.855) (size 0.8) (drill 0.4) (layers "F.Cu" "B.Cu") (free) (net 5))
@@
   (segment (start 110.49 120.0175) (end 113.6405 120.0175) (width 0.6) (layer "F.Cu") (net 6))
   (segment (start 114.913 121.285) (end 116.711324 121.285) (width 0.35) (layer "F.Cu") (net 6))
+  (segment (start 140.335 109.22) (end 139.065 107.95) (width 2) (layer "F.Cu") (net 7))
+  (segment (start 140.335 130.81) (end 140.335 109.22) (width 2) (layer "F.Cu") (net 7))
+  (segment (start 119.57 108.585) (end 129.562 108.585) (width 0.35) (layer "F.Cu") (net 7))
+  (segment (start 139.065 132.08) (end 140.335 130.81) (width 2) (layer "F.Cu") (net 7))
+  (segment (start 139.065 104.14) (end 139.065 102.87) (width 2) (layer "F.Cu") (net 7))
+  (segment (start 139.065 137.16) (end 139.065 132.08) (width 2) (layer "F.Cu") (net 7))
   (segment (start 139.065 107.95) (end 139.065 104.14) (width 2) (layer "F.Cu") (net 7))
-  (segment (start 119.57 108.585) (end 129.562 108.585) (width 0.35) (layer "F.Cu") (net 7))
-  (segment (start 140.335 109.22) (end 139.065 107.95) (width 2) (layer "F.Cu") (net 7))
-  (segment (start 139.065 137.16) (end 139.065 135.89) (width 2) (layer "F.Cu") (net 7))
-  (segment (start 140.335 130.81) (end 140.335 109.22) (width 2) (layer "F.Cu") (net 7))
-  (segment (start 139.065 132.08) (end 140.335 130.81) (width 2) (layer "F.Cu") (net 7))
-  (segment (start 139.065 135.89) (end 139.065 132.08) (width 2) (layer "F.Cu") (net 7))
-  (segment (start 140.97 97.79) (end 142.24 96.52) (width 2) (layer "F.Cu") (net 7))
-  (segment (start 139.065 104.14) (end 139.065 102.87) (width 2) (layer "F.Cu") (net 7))
-  (segment (start 142.24 96.52) (end 150.055 96.52) (width 2) (layer "F.Cu") (net 7))
   (segment (start 129.562 108.585) (end 130.197 109.22) (width 0.35) (layer "F.Cu") (net 7))
   (segment (start 128.248 125.73) (end 128.248 123.855) (width 1) (layer "F.Cu") (net 7))
-  (segment (start 150.055 96.52) (end 158.75 105.215) (width 2) (layer "F.Cu") (net 7))
   (segment (start 128.248 114.3) (end 128.248 115.525) (width 1) (layer "F.Cu") (net 7))
   (via (at 130.175 130.81) (size 0.8) (drill 0.4) (layers "F.Cu" "B.Cu") (free) (net 7))
   (via (at 130.197 127) (size 0.8) (drill 0.4) (layers "F.Cu" "B.Cu") (free) (net 7))
   (via (at 130.175 113.03) (size 0.8) (drill 0.4) (layers "F.Cu" "B.Cu") (free) (net 7))
-  (via (at 140.97 97.79) (size 0.8) (drill 0.4) (layers "F.Cu" "B.Cu") (net 7))
+  (via (at 140.335 102.87) (size 0.8) (drill 0.4) (layers "F.Cu" "B.Cu") (net 7))
   (via (at 130.197 109.22) (size 0.8) (drill 0.4) (layers "F.Cu" "B.Cu") (free) (net 7))
   (via (at 131.467 127) (size 0.8) (drill 0.4) (layers "F.Cu" "B.Cu") (free) (net 7))
-  (via (at 139.7 97.79) (size 0.8) (drill 0.4) (layers "F.Cu" "B.Cu") (free) (net 7))
+  (via (at 140.335 137.16) (size 0.8) (drill 0.4) (layers "F.Cu" "B.Cu") (net 7))
   (via (at 130.175 128.27) (size 0.8) (drill 0.4) (layers "F.Cu" "B.Cu") (free) (net 7))
   (via (at 131.467 113.03) (size 0.8) (drill 0.4) (layers "F.Cu" "B.Cu") (free) (net 7))
@@
   (via (at 130.197 129.54) (size 0.8) (drill 0.4) (layers "F.Cu" "B.Cu") (free) (net 7))
   (via (at 130.175 110.49) (size 0.8) (drill 0.4) (layers "F.Cu" "B.Cu") (free) (net 7))
-  (via (at 138.43 97.79) (size 0.8) (drill 0.4) (layers "F.Cu" "B.Cu") (free) (net 7))
   (via (at 139.065 102.87) (size 0.8) (drill 0.4) (layers "F.Cu" "B.Cu") (free) (net 7))
   (via (at 139.065 135.89) (size 0.8) (drill 0.4) (layers "F.Cu" "B.Cu") (net 7))
+  (segment (start 158.75 105.055) (end 150.215 96.52) (width 2) (layer "B.Cu") (net 7))
+  (segment (start 142.875 96.52) (end 140.97 98.425) (width 2) (layer "B.Cu") (net 7))
+  (segment (start 150.215 96.52) (end 142.875 96.52) (width 2) (layer "B.Cu") (net 7))
   (segment (start 153.035 110.35) (end 153.035 105.41) (width 0.6) (layer "F.Cu") (net 8))
   (segment (start 132.08 114.935) (end 132.08 114.02) (width 0.35) (layer "F.Cu") (net 9))
@@
     (polygon
       (pts
-        (xy 141.605 97.155)
-        (xy 137.795 97.155)
+        (xy 141.605 97.79)
+        (xy 137.16 97.79)
         (xy 129.54 107.95)
         (xy 129.54 113.665)

Commit message: поправил дорожки питания
Routing:
- net VCC: track 71.4 -> 79.8 mm, vias 18 -> 24

Commit message: исправил ошибку в схеме
Connections:
- IC1 pad 1: /SD_LR -> GND
- IC1 pad 3: GND -> /SD_LR
Routing:
- net GND: track 35.0 -> 36.9 mm
- net /SD_LR: track 29.8 -> 30.6 mm
Changed lines of the file:
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@@
       (stroke (width 0.1) (type solid)) (layer "F.Fab"))
     (pad "1" smd rect (at -3.788 -4.875 90) (size 0.45 1.475) (layers "F.Cu" "F.Paste" "F.Mask")
-      (net 16 "/SD_LR") (pinfunction "MODSEL") (pintype "passive"))
+      (net 5 "GND") (pinfunction "MODSEL") (pintype "passive"))
     (pad "2" smd rect (at -3.788 -4.225 90) (size 0.45 1.475) (layers "F.Cu" "F.Paste" "F.Mask")
       (net 16 "/SD_LR") (pinfunction "SD") (pintype "passive"))
     (pad "3" smd rect (at -3.788 -3.575 90) (size 0.45 1.475) (layers "F.Cu" "F.Paste" "F.Mask")
-      (net 5 "GND") (pinfunction "FAULT") (pintype "passive"))
+      (net 16 "/SD_LR") (pinfunction "FAULT") (pintype "passive"))
     (pad "4" smd rect (at -3.788 -2.925 90) (size 0.45 1.475) (layers "F.Cu" "F.Paste" "F.Mask")
       (net 2 "Net-(IC1-RINP)") (pinfunction "RINP") (pintype "passive"))
@@
   (segment (start 106.379 106.045) (end 102.87 106.045) (width 0.35) (layer "F.Cu") (net 1))
   (segment (start 110.744 101.68) (end 106.379 106.045) (width 0.35) (layer "F.Cu") (net 1))
-  (segment (start 120.672 117.09) (end 119.459831 117.09) (width 0.35) (layer "F.Cu") (net 2))
-  (segment (start 114.808 112.438169) (end 114.808 110.744) (width 0.35) (layer "F.Cu") (net 2))
-  (segment (start 119.459831 117.09) (end 114.808 112.438169) (width 0.35) (layer "F.Cu") (net 2))
+  (segment (start 118.909915 117.09) (end 114.808 112.988085) (width 0.35) (layer "F.Cu") (net 2))
   (segment (start 114.808 110.744) (end 110.744 106.68) (width 0.35) (layer "F.Cu") (net 2))
+  (segment (start 120.672 117.09) (end 118.909915 117.09) (width 0.35) (layer "F.Cu") (net 2))
+  (segment (start 114.808 112.988085) (end 114.808 110.744) (width 0.35) (layer "F.Cu") (net 2))
   (segment (start 102.87 110.245) (end 109.799 110.245) (width 0.35) (layer "F.Cu") (net 3))
   (segment (start 109.799 110.245) (end 110.744 109.3) (width 0.35) (layer "F.Cu") (net 3))
-  (segment (start 119.346155 117.74) (end 115.906155 114.3) (width 0.35) (layer "F.Cu") (net 4))
-  (segment (start 120.672 117.74) (end 119.346155 117.74) (width 0.35) (layer "F.Cu") (net 4))
-  (segment (start 115.906155 114.3) (end 110.744 114.3) (width 0.35) (layer "F.Cu") (net 4))
+  (segment (start 118.776538 117.74) (end 115.336538 114.3) (width 0.35) (layer "F.Cu") (net 4))
+  (segment (start 120.672 117.74) (end 118.776538 117.74) (width 0.35) (layer "F.Cu") (net 4))
+  (segment (start 115.336538 114.3) (end 110.744 114.3) (width 0.35) (layer "F.Cu") (net 4))
   (segment (start 128.248 119.69) (end 126.978 119.69) (width 0.35) (layer "F.Cu") (net 5))
   (segment (start 120.672 122.94) (end 121.898 122.94) (width 0.35) (layer "F.Cu") (net 5))
@@
   (segment (start 128.248 121.64) (end 126.978 121.64) (width 0.35) (layer "F.Cu") (net 5))
   (segment (start 120.672 124.24) (end 121.898 124.24) (width 0.35) (layer "F.Cu") (net 5))
-  (segment (start 120.672 116.44) (end 121.898 116.44) (width 0.35) (layer "F.Cu") (net 5))
   (segment (start 120.672 121.64) (end 121.92 121.64) (width 0.35) (layer "F.Cu") (net 5))
   (segment (start 120.672 120.34) (end 121.92 120.34) (width 0.35) (layer "F.Cu") (net 5))
@@
   (segment (start 119.0195 121.2645) (end 119.395 121.64) (width 0.35) (layer "F.Cu") (net 5))
   (segment (start 119.395 121.64) (end 120.672 121.64) (width 0.35) (layer "F.Cu") (net 5))
+  (segment (start 119.38 115.14) (end 122.555 115.14) (width 0.35) (layer "F.Cu") (net 5))
   (segment (start 120.672 120.99) (end 121.92 120.99) (width 0.35) (layer "F.Cu") (net 5))
   (segment (start 119.436 120.34) (end 118.872 120.904) (width 0.35) (layer "F.Cu") (net 5))
@@
   (segment (start 128.248 122.94) (end 130.538 122.94) (width 0.35) (layer "F.Cu") (net 15))
   (segment (start 132.058 124.46) (end 132.058 125.708) (width 0.35) (layer "F.Cu") (net 15))
-  (segment (start 118.273507 115.14) (end 120.672 115.14) (width 0.35) (layer "F.Cu") (net 16))
   (segment (start 116.205 110.3) (end 116.205 110.49) (width 0.35) (layer "F.Cu") (net 16))
+  (segment (start 116.183 111.782) (end 116.183 113.599409) (width 0.35) (layer "F.Cu") (net 16))
+  (segment (start 120.672 116.44) (end 120.672 115.79) (width 0.35) (layer "F.Cu") (net 16))
+  (segment (start 119.023591 116.44) (end 120.672 116.44) (width 0.35) (layer "F.Cu") (net 16))
+  (segment (start 116.205 110.49) (end 116.205 111.76) (width 0.6) (layer "F.Cu") (net 16))
   (segment (start 116.205 111.76) (end 116.183 111.782) (width 0.35) (layer "F.Cu") (net 16))
-  (segment (start 120.672 115.79) (end 120.672 115.14) (width 0.35) (layer "F.Cu") (net 16))
-  (segment (start 116.183 113.049493) (end 118.273507 115.14) (width 0.35) (layer "F.Cu") (net 16))
-  (segment (start 116.205 110.49) (end 116.205 111.76) (width 0.6) (layer "F.Cu") (net 16))
-  (segment (start 116.183 111.782) (end 116.183 113.049493) (width 0.35) (layer "F.Cu") (net 16))
+  (segment (start 116.183 113.599409) (end 119.023591 116.44) (width 0.35) (layer "F.Cu") (net 16))
   (segment (start 117.92 108.585) (end 116.205 110.3) (width 0.35) (layer "F.Cu") (net 16))
   (via (at 116.205 110.49) (size 1) (drill 0.4) (layers "F.Cu" "B.Cu") (net 16))
