File: tpa3116_amplifier_board.kicad_pcb (KiCad board)
At the start: 2 copper layers, 73 x 54.6 mm, 58 parts, among them IC1 TPA3116D2QDADRQ1, J1 control, J2 control, J3 output_right, J4 output_left, J5 power_supply, J6 power_supply

Commit message: Добавил надписи
Routing:
- net /SD_LR: track 29.7 -> 30.6 mm
Other:
- board size 73 x 54.6 mm -> 72.4 x 54.6 mm

Commit message: исправил ошибку в схеме, добавил разъемы
Parts:
- removed C28: 10n, Capacitor_SMD:C_0603_1608Metric
- removed J5, J6: power_supply, Connector_Wire:SolderWire-1sqmm_1x02_P5.4mm_D1.4mm_OD2.7mm
- C14: value 220n -> 35v 470u; footprint Capacitor_SMD:C_0603_1608Metric -> Capacitor_THT:CP_Radial_D10.0mm_P5.00mm
- C16: value 35v 470u -> 680n; footprint Capacitor_THT:CP_Radial_D10.0mm_P5.00mm -> Capacitor_THT:C_Rect_L7.0mm_W4.5mm_P5.00mm
- C17, C18, C19: value 470n -> 680n
- C20: value 470n -> 1n; footprint Capacitor_THT:C_Rect_L7.0mm_W4.5mm_P5.00mm -> Capacitor_SMD:C_0603_1608Metric
- C24: value 1n -> 10n
- C5: value -- -> 1u; footprint Capacitor_SMD:C_0603_1608Metric -> Capacitor_SMD:C_0805_2012Metric
- C6: value 1u -> 1n; footprint Capacitor_SMD:C_0805_2012Metric -> Capacitor_SMD:C_0603_1608Metric
- C8: value 1n -> 220n
- J1, J2: footprint Connector_Wire:SolderWire-0.25sqmm_1x04_P4.2mm_D0.65mm_OD1.7mm -> Connector_JST:JST_EH_B4B-EH-A_1x04_P2.50mm_Vertical
- J3: value output_right -> power_supply; footprint Connector_Wire:SolderWire-1sqmm_1x02_P5.4mm_D1.4mm_OD2.7mm -> Connector_JST:JST_VH_B2P-VH-B_1x02_P3.96mm_Vertical
- J4: value output_left -> control; footprint Connector_Wire:SolderWire-1sqmm_1x02_P5.4mm_D1.4mm_OD2.7mm -> Connector_JST:JST_VH_B4P-VH-B_1x04_P3.96mm_Vertical
- L1, L4: value 22u -> 10u
- moved C20 40.8 mm to (153.7, 95.7), turned to -90 degrees
- moved C16 38.6 mm to (153.7, 104.7), turned to 90 degrees
- moved C24 33.0 mm to (152.4, 109.2)
- moved C17 20.9 mm to (145.4, 113.0), turned to -90 degrees
- moved C8 20.3 mm to (118.7, 130.2), turned to 180 degrees
- moved C10 18.2 mm to (126.4, 113.7), turned to 90 degrees
- moved C6 18.2 mm to (118.7, 127.6), turned to 180 degrees
- moved C9 17.8 mm to (118.7, 109.9)
- moved C19 17.5 mm to (153.7, 140.3), turned to 90 degrees
- moved C22 17.5 mm to (145.4, 130.9), turned to 90 degrees
- moved C23 15.3 mm to (153.7, 144.1), turned to -90 degrees
- moved C18 14.6 mm to (145.4, 122.0), turned to -90 degrees
- moved C14 14.2 mm to (129.1, 140.3), turned to 0 degrees
- moved R11 13.4 mm to (149.2, 130.8), turned to 90 degrees
- moved C25 10.5 mm to (151.8, 114.7), turned to -90 degrees
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Connections:
- C10 pad 1: VCC -> Net-(IC1-OUTPR)
- C10 pad 2: GND -> Net-(IC1-BSPR)
- C11 pad 1: Net-(IC1-OUTPR) -> Net-(IC1-OUTNR)
- C11 pad 2: Net-(IC1-BSPR) -> Net-(IC1-BSNR)
- C12 pad 1: Net-(IC1-OUTNR) -> Net-(IC1-OUTPL)
- C12 pad 2: Net-(IC1-BSNR) -> Net-(IC1-BSPL)
- C13 pad 1: Net-(IC1-OUTPL) -> Net-(IC1-OUTNL)
- C13 pad 2: Net-(IC1-BSPL) -> Net-(IC1-BSNL)
- C14 pad 1: Net-(IC1-OUTNL) -> VCC
- C14 pad 2: Net-(IC1-BSNL) -> GND
- C16 pad 1: VCC -> GND
- C16 pad 2: GND -> Net-(J4-Pin_4)
- C17 pad 1: GND -> Net-(J4-Pin_3)
- C17 pad 2: Net-(J3-Pin_1) -> GND
- C18 pad 1: Net-(J3-Pin_2) -> GND
- C18 pad 2: GND -> Net-(J4-Pin_2)
- C19 pad 1: GND -> Net-(J4-Pin_1)
- C19 pad 2: Net-(J4-Pin_1) -> GND
- C20 pad 1: Net-(J4-Pin_2) -> GND
- C20 pad 2: GND -> Net-(J4-Pin_4)
- C21 pad 1: GND -> Net-(J4-Pin_3)
- C21 pad 2: Net-(J3-Pin_1) -> GND
- C22 pad 1: Net-(J3-Pin_2) -> GND
- C22 pad 2: GND -> Net-(J4-Pin_2)
- C23 pad 1: GND -> Net-(J4-Pin_1)
- C23 pad 2: Net-(J4-Pin_1) -> GND
- C24 pad 1: Net-(J4-Pin_2) -> Net-(J4-Pin_4)
- C24 pad 2: GND -> Net-(C24-Pad2)
- C25 pad 1: GND -> Net-(J4-Pin_3)
- C26 pad 1: GND -> Net-(J4-Pin_2)
- C27 pad 1: GND -> Net-(J4-Pin_1)
- C6 pad 1: GND -> VCC
- C6 pad 2: Net-(IC1-GVDD) -> GND
- C7 pad 1: VCC -> GND
- C7 pad 2: GND -> VCC
- C8 pad 1: GND -> VCC
- C8 pad 2: VCC -> GND
- IC1 pad 1: /SD_LR -> GND
- IC1 pad 3: GND -> /SD_LR
- J3 pad 1: Net-(J3-Pin_1) -> GND
- J3 pad 2: Net-(J3-Pin_2) -> VCC
- L1 pad 2: Net-(J3-Pin_1) -> Net-(J4-Pin_4)
- L2 pad 2: Net-(J3-Pin_2) -> Net-(J4-Pin_3)
- L3 pad 2: Net-(J4-Pin_1) -> Net-(J4-Pin_2)
- L4 pad 2: Net-(J4-Pin_2) -> Net-(J4-Pin_1)
- R10 pad 1: Net-(J4-Pin_1) -> GND
- R10 pad 2: Net-(C27-Pad2) -> Net-(C26-Pad2)
- R11 pad 1: Net-(J4-Pin_2) -> GND
- R11 pad 2: Net-(C28-Pad2) -> Net-(C27-Pad2)
- R8 pad 1: Net-(J3-Pin_1) -> GND
- R8 pad 2: Net-(C25-Pad2) -> Net-(C24-Pad2)
- R9 pad 1: Net-(J3-Pin_2) -> GND
- R9 pad 2: Net-(C26-Pad2) -> Net-(C25-Pad2)
Routing:
- net Net-(J4-Pin_4): track 0.00 -> 45.5 mm
- net Net-(J3-Pin_1): track 33.1 -> 0.00 mm
- net Net-(J4-Pin_3): track 0.00 -> 28.6 mm
- net Net-(J3-Pin_2): track 28.0 -> 0.00 mm
- net VCC: track 103.8 -> 120.5 mm, vias 24 -> 16
- net Net-(J4-Pin_2): track 33.1 -> 21.9 mm
- net Net-(IC1-OUTPL): track 20.7 -> 12.2 mm
- net Net-(IC1-OUTNR): track 19.1 -> 11.8 mm
- net Net-(C24-Pad2): track 0.00 -> 3.20 mm
- net Net-(J4-Pin_1): track 31.5 -> 28.7 mm
- net GND: track 31.6 -> 28.9 mm, vias 134 -> 97
- net /R+: track 9.31 -> 11.9 mm
- net /L-: track 21.4 -> 23.7 mm
- net Net-(C28-Pad2): track 2.26 -> 0.00 mm
- net /SD_LR: track 30.6 -> 32.7 mm
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Other:
- board size 72.4 x 54.6 mm -> 73 x 54.6 mm
- board text added: "fault"
- board text removed: "sd_lr"
