File: tpa3116_amplifier_board.kicad_sch (KiCad schematic)
At the start: 41 parts, among them IC1 TPA3116D2QDADRQ1, J1 power_supply, J2 Conn_01x04, J3 power_supply, J4 output_right

Commit message: исправил ошибку в схеме
Connections:
- net GND: now also IC1.1 (MODSEL); no longer IC1.3 (FAULT)
- net SD_LR: now also IC1.3 (FAULT); no longer IC1.1 (MODSEL)
Changed lines of the file:
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@@
   (junction (at 109.22 116.84) (diameter 0) (color 0 0 0 0)
   )
-  (junction (at 106.68 83.82) (diameter 0) (color 0 0 0 0)
+  (junction (at 106.68 86.36) (diameter 0) (color 0 0 0 0)
   )
   (junction (at 66.04 78.74) (diameter 0) (color 0 0 0 0)
@@
     (stroke (width 0) (type default))
   )
-  (wire (pts (xy 106.68 77.47) (xy 106.68 83.82))
+  (wire (pts (xy 106.68 77.47) (xy 106.68 86.36))
     (stroke (width 0) (type default))
   )
@@
     (stroke (width 0) (type default))
   )
+  (wire (pts (xy 104.14 83.82) (xy 114.3 83.82))
+    (stroke (width 0) (type default))
+  )
   (wire (pts (xy 49.53 104.14) (xy 114.3 104.14))
     (stroke (width 0) (type default))
@@
     (stroke (width 0) (type default))
   )
-  (wire (pts (xy 106.68 83.82) (xy 106.68 86.36))
-    (stroke (width 0) (type default))
-  )
   (wire (pts (xy 166.37 83.82) (xy 179.07 83.82))
     (stroke (width 0) (type default))
@@
     (stroke (width 0) (type default))
   )
+  (wire (pts (xy 106.68 88.9) (xy 106.68 86.36))
+    (stroke (width 0) (type default))
+  )
   (wire (pts (xy 238.76 81.28) (xy 252.73 81.28))
     (stroke (width 0) (type default))
@@
     (stroke (width 0) (type default))
   )
+  (wire (pts (xy 114.3 88.9) (xy 106.68 88.9))
+    (stroke (width 0) (type default))
+  )
   (wire (pts (xy 196.85 114.3) (xy 196.85 124.46))
     (stroke (width 0) (type default))
@@
     (stroke (width 0) (type default))
   )
-  (wire (pts (xy 97.79 88.9) (xy 114.3 88.9))
-    (stroke (width 0) (type default))
-  )
   (wire (pts (xy 179.07 88.9) (xy 173.99 88.9))
     (stroke (width 0) (type default))
@@
     (stroke (width 0) (type default))
   )
-  (wire (pts (xy 90.17 83.82) (xy 106.68 83.82))
+  (wire (pts (xy 88.9 86.36) (xy 106.68 86.36))
     (stroke (width 0) (type default))
   )
@@
   )
   (wire (pts (xy 157.48 83.82) (xy 166.37 83.82))
-    (stroke (width 0) (type default))
-  )
-  (wire (pts (xy 114.3 83.82) (xy 106.68 83.82))
     (stroke (width 0) (type default))
   )
@@
     (effects (font (size 1.27 1.27)) (justify left bottom))
   )
-  (label "SD_LR" (at 90.17 83.82 0) (fields_autoplaced)
+  (label "SD_LR" (at 88.9 86.36 0) (fields_autoplaced)
     (effects (font (size 1.27 1.27)) (justify left bottom))
   )
@@
     )
   )
-  (symbol (lib_id "power:GND") (at 97.79 88.9 270) (unit 1)
-    (in_bom yes) (on_board yes) (dnp no)
-    (property "Reference" "#PWR05" (at 91.44 88.9 0)
-      (effects (font (size 1.27 1.27)) hide)
-    )
-    (property "Value" "GND" (at 93.98 88.9 90)
+  (symbol (lib_id "power:GND") (at 104.14 83.82 270) (unit 1)
+    (in_bom yes) (on_board yes) (dnp no)
+    (property "Reference" "#PWR05" (at 97.79 83.82 0)
+      (effects (font (size 1.27 1.27)) hide)
+    )
+    (property "Value" "GND" (at 100.33 83.82 90)
       (effects (font (size 1.27 1.27)) (justify right))
     )
-    (property "Footprint" "" (at 97.79 88.9 0)
-      (effects (font (size 1.27 1.27)) hide)
-    )
-    (property "Datasheet" "" (at 97.79 88.9 0)
-      (effects (font (size 1.27 1.27)) hide)
-    )
+    (property "Footprint" "" (at 104.14 83.82 0)
+      (effects (font (size 1.27 1.27)) hide)
+    )
+    (property "Datasheet" "" (at 104.14 83.82 0)
+      (effects (font (size 1.27 1.27)) hide)
+    )
