File: tpa3116_amplifier_board.kicad_sch (KiCad schematic)
At the start: 58 parts, among them IC1 TPA3116D2QDADRQ1, J1 control, J2 control, J3 output_right, J4 output_left, J5 power_supply, J6 power_supply

Commit message: исправил ошибку в схеме, добавил разъемы
Parts:
- removed C5: --, Capacitor_SMD:C_0603_1608Metric, symbol Device:C
- removed J3: output_right, Connector_Wire:SolderWire-1sqmm_1x02_P5.4mm_D1.4mm_OD2.7mm, symbol Connector_Generic:Conn_01x02
- removed J4: output_left, Connector_Wire:SolderWire-1sqmm_1x02_P5.4mm_D1.4mm_OD2.7mm, symbol Connector_Generic:Conn_01x02
- removed J6: power_supply, Connector_Wire:SolderWire-1sqmm_1x02_P5.4mm_D1.4mm_OD2.7mm, symbol Connector_Generic:Conn_01x02
- added J4: control, Connector_JST:JST_VH_B4P-VH-B_1x04_P3.96mm_Vertical, symbol Connector_Generic:Conn_01x04
- C16: renamed from C17; value 470n -> 680n
- C17: renamed from C18; value 470n -> 680n
- C18: renamed from C19; value 470n -> 680n
- C19: renamed from C20; value 470n -> 680n
- J1, J2: footprint Connector_Wire:SolderWire-0.25sqmm_1x04_P4.2mm_D0.65mm_OD1.7mm -> Connector_JST:JST_EH_B4B-EH-A_1x04_P2.50mm_Vertical
- J3: renamed from J5; footprint Connector_Wire:SolderWire-1sqmm_1x02_P5.4mm_D1.4mm_OD2.7mm -> Connector_JST:JST_VH_B2P-VH-B_1x02_P3.96mm_Vertical
- L1, L4: value 22u -> 10u
- renumbered C11 to C10, C12 to C11, C13 to C12, C14 to C13, C15 to C14, C16 to C15, C21 to C20, C22 to C21, C23 to C22, C24 to C23, C25 to C24, C26 to C25, C27 to C26, C28 to C27, C6 to C5, C7 to C6, C8 to C7, C9 to C8, C10 to C9
Connections:
- net GND: now also IC1.1 (MODSEL), R10.1, R11.1, R8.1, R9.1; no longer C24.1, C25.1, C26.1, C27.1, IC1.3 (FAULT)
- net SD_LR: now also IC1.3 (FAULT); no longer IC1.1 (MODSEL)
- net at C19.1, C23.1, L4.2: now also C27.1, J4.1 (Pin_1); no longer R11.1
- net at C16.2, C20.2, L1.2: now also C24.1, J4.4 (Pin_4); no longer R8.1
- net at C17.1, C21.1, L2.2: now also C25.1, J4.3 (Pin_3); no longer R9.1
- net at C18.2, C22.2, L3.2: now also C26.1, J4.2 (Pin_2); no longer R10.1
Other:
- moved on the sheet: C24, C25, C26, C27, R10, R11, R8, R9
